Commit message: add fr3 support demo 5/6 and add demo 09

File: agimus_demo_05_pick_and_place/urdf/demo.urdf.xacro (robot description, xacro)
@@ -1,5 +1,6 @@
 <?xml version='1.0' encoding='utf-8'?>
 <robot xmlns:xacro="http://www.ros.org/wiki/xacro" name="panda">
-  <xacro:include filename="$(find franka_description)/robots/fer/fer.urdf.xacro">
+  <xacro:arg name="arm_id" default="fer" />
+  <xacro:include filename="$(find franka_description)/robots/$(arg arm_id)/$(arg arm_id).urdf.xacro">
     <!-- <xacro:arg name="with_sc" value="True" /> -->
   </xacro:include>

File: agimus_demo_05_pick_and_place/urdf/support.urdf.xacro (robot description, xacro)
@@ -6,5 +6,5 @@
         <mass value="200" />
         <origin xyz="0 0 0.45" />
-        <inertia ixx="50" ixy="0" ixz="0" iyy="50" iyz="0" izz="50" />
+        <!-- <inertia ixx="50" ixy="0" ixz="0" iyy="50" iyz="0" izz="50" /> -->
       </inertial>
       <visual>

File: agimus_demo_06_regrasp/urdf/support.urdf.xacro (robot description, xacro)
@@ -6,5 +6,5 @@
         <mass value="200" />
         <origin xyz="0 0 0.45" />
-        <inertia ixx="50" ixy="0" ixz="0" iyy="50" iyz="0" izz="50" />
+        <inertia ixx="0" ixy="0" ixz="0" iyy="0" iyz="0" izz="0" />
       </inertial>
       <visual>
@@ -245,5 +245,5 @@
       <parent link="support_link" />
       <child link="pedestal" />
-    </joint>
+    </joint>v
     <joint name="foam_block_joint" type="fixed">
       <origin xyz="0.0 -0.08 0.75" />

File: agimus_demo_09_glue_spreading/urdf/demo.urdf.xacro (robot description, xacro)
@@ -5,9 +5,8 @@
     <!-- <xacro:arg name="with_sc" value="True" /> -->
   </xacro:include>
-  <xacro:include filename="$(find agimus_demo_06_regrasp)/urdf/support.urdf.xacro"/>
-  <xacro:support/>
-  <joint name="attach_robot_joint" type="fixed">
-    <parent link="robot_attachment_link" />
-    <child link="base" />
+  <xacro:include filename="$(find agimus_demo_09_glue_spreading)/urdf/table.urdf.xacro"/>
+  <xacro:table parent_link="world" child_link="base">
+    <origin xyz="0 0 0.68" rpy="0 0 0"/>
+  </xacro:table>
 </joint>
 </robot>
