Commit message: [pre-commit.ci] auto fixes from pre-commit.com hooks
for more information, see https://pre-commit.ci

File: agimus_demo_09_glue_spreading/urdf/plate.urdf.xacro (robot description, xacro)
@@ -22,5 +22,5 @@
       parent_link: Le maillon auquel attacher cette bordure
       size_x, size_y, size_z: Dimensions de la boîte de la bordure
-      *origin: Bloc <origin> pour la position relative au parent
+      *origin: Block <origin> pour la position relative au parent
   -->
   <xacro:macro name="single_border" params="name parent_link size_x size_y size_z *origin">
@@ -46,5 +46,5 @@
     Cette macro génère une plaque et appelle 4 fois la macro single_border.
     Params:
-      name: Préfixe pour tous les liens et joints
+      name: Préfixe pour tous les lines et joints
       *origin: Position de la plaque par rapport au parent
   -->
@@ -60,5 +60,5 @@
       </collision>
     </link>
-    <!-- Instanciation des 4 bordures en appelant la macro single_border -->
+    <!-- Instantiation des 4 bordures en appelant la macro single_border -->
     <!-- Bordure Avant (+X) -->
     <xacro:single_border name="${name}_border_front" parent_link="${name}_base_link"
